File: hardware/mpcie-msata.kicad_pcb (KiCad board)
At the start: 4 copper layers, 100 x 85 mm, 202 parts, among them J102 TNG-Power-BTM, J103 TNG-Power-TOP, J104 TNG-Data-BTM, J105 TNG-Data-TOP, J201 Mini-PCIE, J202 SIM8060, J301 Mini-SATA, P101 Debug, P102 PE, Q301 40MHz, SW101 BOOT, U101 USB2514B, U102 LD1117, U103 TPS7A7002, U104 STM32F070CBT6, U105 82400152, U201 LM813, U301 TUSB9261PVP, U302 TLV71211DBVR, U303 AP7333-18SAG-7, U304 AT25DF011-SSHN-T, X101 24MHz, X102 TBD

Commit message: nearly completely routed
Parts:
- removed the Fiducial_Mark at (152.4, 56.0)
- added Fiducial_Mark: VAL**, kicad-libraries:Fiducial_Mark, F.Cu at (59.5, 133.9)
- added Fiducial_Mark: VAL**, kicad-libraries:Fiducial_Mark, F.Cu at (154.4, 54.0)
- C208, R302, R303: moved to F.Cu
- C322, R106, R111, R117: moved to B.Cu
- D102: value LED -> blue
- Q301: footprint kicad-libraries:CRYSTAL_3225 -> kicad-libraries:CRYSTAL_3225_4
- moved R111 97.8 mm to (117.1, 60.3), turned to 90 degrees
- moved R106 97.4 mm to (117.1, 62.2), turned to 270 degrees
- moved R117 96.1 mm to (118.1, 60.3), turned to 90 degrees
- moved P101 7.67 mm to (110.4, 65.4)
- moved R306 5.34 mm to (127.5, 86.2)
- moved C117 3.70 mm to (133.5, 56.6), turned to 90 degrees
- moved R110 3.65 mm to (135.1, 65.3), turned to 0 degrees
- moved C327 3.21 mm to (137.1, 78.8), turned to 180 degrees
- moved C322 3.19 mm to (132.2, 78.6), turned to 180 degrees
- moved R305 2.93 mm to (132.2, 90.2), turned to 180 degrees
- moved R121 2.62 mm to (118.6, 57.4), turned to 270 degrees
- moved C340 2.17 mm to (128.1, 75.5)
- moved C319 2.08 mm to (138.3, 76.0), turned to 270 degrees
- moved R124 2.05 mm to (140.8, 97.8), turned to 270 degrees
- moved C318 1.92 mm to (134.0, 79.6)
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Connections:
- net Net-(C143-Pad1) renamed LDO-IN
- C347 pad 2: VDD_3P3V -> 3V3
- J301 pad 49: (no net) -> MSATA_ACTIVITY_LED
- R201 pad 2: (no net) -> MPCIE_PPS
- R203 pad 1: MPCIE_#RESET -> Net-(C201-Pad1)
- R203 pad 2: +3.3VP -> MPCIE_#RESET
- R205 pad 2: +3.3VP -> 3V3
- R206 pad 2: +3.3VP -> 3V3
- R311 pad 1: VDD_3P3V -> 3V3
- R312 pad 1: VDD_3P3V -> 3V3
- R313 pad 2: VDD_3P3V -> 3V3
- RP201 pad 1: (no net) -> MPCIE_LED_WWAN
- RP201 pad 2: (no net) -> MPCIE_LED_WIFI
- RP201 pad 4: (no net) -> MPCIE_LED_WPAN
- RP202 pad 1: Net-(RP202-Pad1) -> (no net)
- RP202 pad 4: (no net) -> Net-(RP202-Pad4)
- RP202 pad 5: (no net) -> LM813_BT_WAKE_HOST
- RP202 pad 6: (no net) -> LM813_LED_BT
- RP202 pad 7: (no net) -> LM813_LED_WL
- U104 pad 10: (no net) -> LM813_LED_WL
- U104 pad 11: (no net) -> LM813_WLAN_DIS
- U104 pad 12: (no net) -> MSATA_RX
- U104 pad 13: Net-(D102-Pad2) -> MSATA_TX
- U104 pad 14: (no net) -> MSATA_SPI_CS
- U104 pad 15: (no net) -> MSATA_SPI_CLK
- U104 pad 16: (no net) -> MSATA_SPI_DI
- U104 pad 17: (no net) -> MSATA_SPI_DO
- U104 pad 18: Net-(P101-Pad1) -> MPCIE_#DISABLE
- U104 pad 19: (no net) -> MPCIE_#RESET
- U104 pad 2: (no net) -> LM813_BT_DIS
- U104 pad 20: (no net) -> MPCIE_LED_WWAN
- U104 pad 21: (no net) -> MPCIE_LED_WIFI
- U104 pad 22: (no net) -> MPCIE_LED_WPAN
- U104 pad 25: USB_RESET -> MPCIE_PPS
- U104 pad 26: (no net) -> MSATA_EN
- U104 pad 27: (no net) -> MSATA_ACTIVITY_LED
- U104 pad 3: (no net) -> LM813_LED_BT
- U104 pad 34: (no net) -> USB_RESET
- U104 pad 37: (no net) -> Net-(D102-Pad2)
- U104 pad 4: (no net) -> LM813_BT_WAKE_HOST
- U104 pad 40: (no net) -> Net-(P101-Pad1)
- U104 pad 46: (no net) -> LM813_EN
- U201 pad 1: Net-(RP202-Pad1) -> Net-(RP202-Pad4)
- U304 pad 8: VDD_3P3V -> 3V3
Routing:
- net GND: track 93.0 -> 369.1 mm, vias 36 -> 274
- net 3V3: track 19.1 -> 209.5 mm, vias 13 -> 31
- net 5V: track 0.00 -> 162.2 mm, vias 0 -> 12
- net +3.3VP: track 0.00 -> 108.8 mm, vias 0 -> 15
- net Net-(C301-Pad2): track 0.00 -> 95.0 mm, vias 0 -> 8
- net Net-(C201-Pad1): track 0.00 -> 76.5 mm, vias 0 -> 9
- net Earth: track 170.1 -> 93.8 mm
- net +1.1V: track 0.00 -> 69.7 mm, vias 0 -> 11
- net MSATA_SPI_DI: track 0.00 -> 69.1 mm, vias 0 -> 2
- net MSATA_SPI_CLK: track 0.00 -> 68.8 mm, vias 0 -> 2
- net MSATA_SPI_CS: track 0.00 -> 67.6 mm, vias 0 -> 2
- net MSATA_SPI_DO: track 0.00 -> 64.8 mm, vias 0 -> 2
- net 5V-STACK: track 101.0 -> 162.2 mm, vias 0 -> 5
- net MPCIE_#DISABLE: track 0.00 -> 54.5 mm
- net MPCIE_PPS: track 0.00 -> 54.2 mm, vias 0 -> 3
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- added copper zone on B.Cu, net GND
- added copper zone on F.Cu, net GND
- added copper zone on GND, net GND
- added copper zone on F.Cu, net LDO-IN
Other:
- board text added: "Mini PCI-E"
- board text added: "Mini SATA"

Commit message: routing improvement
Parts:
- moved C125 1.90 mm to (139.9, 69.7)
- moved C346 1.67 mm to (141.2, 74.5)
- moved C344 0.85 mm to (141.3, 72.2), turned to 180 degrees
- moved C317 0.81 mm to (140.4, 77.8), turned to 180 degrees
Connections:
- net Net-(C201-Pad1) renamed 3V3-MPCIE
- net Net-(C301-Pad2) renamed 3V3-MSATA
- J104 pad 38: (no net) -> Net-(J104-Pad38)
- J105 pad 29: (no net) -> Net-(J104-Pad38)
- J201 pad MNT: (no net) -> GND
- J301 pad MNT: (no net) -> GND
Routing:
- net 3V3-MSATA: track 95.0 -> 118.7 mm
- net GND: track 369.1 -> 389.3 mm, vias 274 -> 285
- net PWR-VCC: track 49.4 -> 67.6 mm
- net 5V-STACK: track 162.2 -> 175.0 mm, vias 5 -> 20
- net Net-(J104-Pad14): track 0.00 -> 7.29 mm, vias 0 -> 1
- net Net-(J104-Pad20): track 0.00 -> 7.23 mm, vias 0 -> 1
- net Net-(J104-Pad28): track 0.00 -> 7.17 mm, vias 0 -> 1
- net Net-(J104-Pad36): track 0.00 -> 7.11 mm, vias 0 -> 1
- net Net-(J104-Pad22): track 0.00 -> 6.88 mm, vias 0 -> 1
- net Net-(J104-Pad38): track 0.00 -> 6.81 mm, vias 0 -> 1
- net Net-(J104-Pad30): track 0.00 -> 6.78 mm, vias 0 -> 1
- net Net-(J104-Pad12): track 0.00 -> 6.76 mm, vias 0 -> 1
- net Net-(C328-Pad1): track 4.80 -> 8.70 mm, vias 0 -> 2
- net +3.3VP: track 108.8 -> 105.2 mm, vias 15 -> 14
- net 3V3: track 209.5 -> 212.6 mm
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- added copper zone on VCC, net +3.3VP
- added copper zone on VCC, net 3V3
- added copper zone on VCC, net 3V3-MPCIE
- added copper zone on VCC, net 3V3-MSATA
- added copper zone on B.Cu, net Earth
- added copper zone on B.Cu, net PWR-GND
- added copper zone on B.Cu, net PWR-VCC
- removed copper zone on B.Cu, net STACKPWR
