File: hardware/mpcie-msata.kicad_pcb (KiCad board)
At the start: 4 copper layers, 100 x 85 mm, 203 parts, among them J102 TNG-Power-BTM, J103 TNG-Power-TOP, J104 TNG-Data-BTM, J105 TNG-Data-TOP, J201 Mini-PCIE, J202 SIM8060, J301 Mini-SATA, P101 Debug, P102 PE, Q301 40MHz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

Commit message: add fiducials
Parts:
- added Fiducial_Mark: VAL**, kicad-libraries:Fiducial_Mark, B.Cu at (60.5, 57.0)
- added Fiducial_Mark: VAL**, kicad-libraries:Fiducial_Mark, F.Cu at (60.5, 57.0)

Commit message: add clamp
Routing:
- net Earth: track 93.8 -> 94.1 mm, vias 25 -> 20
Changed lines of the file:
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@@
     (thickness 1.6)
     (drawings 15)
-    (tracks 2821)
+    (tracks 2816)
     (zones 0)
     (modules 205)
@@
   (page A4)
   (layers
-    (0 F.Cu power)
+    (0 F.Cu power hide)
     (1 GND power hide)
     (2 VCC power hide)
@@
     (aux_axis_origin 57.45 50.95)
     (grid_origin 57.45 50.95)
-    (visible_elements FFFEFFFF)
+    (visible_elements FFFFFFFF)
     (pcbplotparams
       (layerselection 0x010fc_ffffffff)
@@
     (diff_pair_gap 0.3)
   )
+  (module kicad-libraries:PE_Hook (layer F.Cu)
+    (at 155.95 128.05)
+    (fp_text reference P102 (at 0 0.5) (layer F.Fab)
+      (effects (font (size 0.15 0.15) (thickness 0.0375)))
+    )
+    (fp_text value PE (at 0 -0.5) (layer F.Fab)
+      (effects (font (size 0.15 0.15) (thickness 0.0375)))
+    )
+    (pad 1 thru_hole oval (at -0.15 -1.075) (size 1 2) (drill oval 0.45 1.2) (layers *.Cu *.Mask)
+      (net 1 Earth))
+    (pad 1 thru_hole oval (at -0.15 5.925) (size 1 2) (drill oval 0.45 1.2) (layers *.Cu *.Mask)
+      (net 1 Earth))
+    (pad 1 smd rect (at 0 0) (size 3 15.85) (layers F.Cu)
+      (net 1 Earth))
+    (model Connectors_TF/PE_Hook.wrl
+      (at (xyz 0 0 0))
+      (scale (xyz 1 1 1))
+      (rotate (xyz 0 0 0))
+    )
+  )
   (module kicad-libraries:Fiducial_Mark (layer B.Cu)
     (at 60.45 56.95)
@@
     )
   )
-  (module kicad-libraries:PE_Hook (layer F.Cu)
-    (at 155.95 128.05)
-    (fp_text reference P102 (at 0 0.5) (layer F.Fab)
-      (effects (font (size 0.15 0.15) (thickness 0.0375)))
-    )
-    (fp_text value PE (at 0 -0.5) (layer F.Fab)
-      (effects (font (size 0.15 0.15) (thickness 0.0375)))
-    )
-    (pad 1 smd rect (at 0 0) (size 3 15.85) (layers F.Cu F.Paste F.Mask)
-      (net 1 Earth))
-    (pad 1 smd rect (at 0 0) (size 3 15.85) (layers B.Cu B.Paste B.Mask)
-      (net 1 Earth))
-  )
   (module R0402F (layer F.Cu)
     (at 68 54.6 180)
@@
   (segment (start 153.95 124.525) (end 152.1687 122.7437) (width 0.7) (layer F.Cu) (net 1))
   (segment (start 152.1687 122.7437) (end 149.725 122.7437) (width 0.7) (layer F.Cu) (net 1) (status 800000))
-  (via (at 155.95 128.05) (size 0.7) (drill 0.25) (layers F.Cu B.Cu) (net 1))
-  (via (at 155.95 127.05) (size 0.7) (drill 0.25) (layers F.Cu B.Cu) (net 1))
   (segment (start 155.95 128.05) (end 155.95 127.05) (width 0.2) (layer F.Cu) (net 1))
-  (via (at 155.95 126.05) (size 0.7) (drill 0.25) (layers F.Cu B.Cu) (net 1))
   (segment (start 155.95 127.05) (end 155.95 126.05) (width 0.2) (layer B.Cu) (net 1))
   (via (at 155.95 125.05) (size 0.7) (drill 0.25) (layers F.Cu B.Cu) (net 1))
@@
   (via (at 155.95 132.05) (size 0.7) (drill 0.25) (layers F.Cu B.Cu) (net 1))
   (segment (start 155.95 131.05) (end 155.95 132.05) (width 0.2) (layer F.Cu) (net 1))
-  (via (at 155.95 133.05) (size 0.7) (drill 0.25) (layers F.Cu B.Cu) (net 1))
   (segment (start 155.95 132.05) (end 155.95 133.05) (width 0.2) (layer B.Cu) (net 1))
-  (via (at 155.95 134.05) (size 0.7) (drill 0.25) (layers F.Cu B.Cu) (net 1))
   (segment (start 155.95 128.05) (end 155.95 134.05) (width 0.2) (layer F.Cu) (net 1))
-  (via (at 155.95 135.05) (size 0.7) (drill 0.25) (layers F.Cu B.Cu) (net 1))
-  (segment (start 155.95 128.05) (end 155.95 135.05) (width 0.2) (layer B.Cu) (net 1))
   (segment (start 155.95 128.05) (end 152.25 128.05) (width 1) (layer F.Cu) (net 1))
   (via (at 146.95 120.35) (size 0.7) (drill 0.25) (layers F.Cu B.Cu) (net 1))
@@
   (segment (start 149.725 123.55) (end 147.95 123.55) (width 0.5) (layer B.Cu) (net 1))
   (segment (start 147.95 123.55) (end 149.7 123.55) (width 0.5) (layer F.Cu) (net 1))
+  (via (at 155.95 135.34999) (size 0.7) (drill 0.25) (layers F.Cu B.Cu) (net 1))
+  (segment (start 155.95 128.05) (end 155.95 135.34999) (width 0.2) (layer B.Cu) (net 1))
   (segment (start 137.758508 65.608508) (end 137.8 65.65) (width 0.2) (layer B.Cu) (net 2))
   (segment (start 136.55 65.35) (end 136.808508 65.608508) (width 0.2) (layer B.Cu) (net 2))
